Commit message: ECNG3020: First Modifications

File: crazyflie_gazebo/models/rotors_description/urdf/crazyflie.xacro (robot description, xacro)
@@ -25,12 +25,12 @@
   <xacro:property name="rotor_offset_top" value="0.0125" /> <!-- [m] -->
   <xacro:property name="radius_rotor" value="0.0225" /> <!-- [m] -->
-  <xacro:property name="motor_constant" value="1.2819184e-8" /> <!-- [kg.m/s^2] -->
+  <xacro:property name="motor_constant" value="1.28192e-08" /> <!-- [kg.m/s^2] -->
   <xacro:property name="moment_constant" value="0.005964552" /> <!-- [m] -->
   <xacro:property name="time_constant_up" value="0.0125" /> <!-- [s] -->
   <xacro:property name="time_constant_down" value="0.025" /> <!-- [s] -->
-  <xacro:property name="max_rot_velocity" value="3052" /> <!-- [rad/s] -->
-  <xacro:property name="rotor_drag_coefficient" value="9.1785e-7" />
+  <xacro:property name="max_rot_velocity" value="2618" /> <!-- [rad/s] -->
+  <xacro:property name="rotor_drag_coefficient" value="8.06428e-05" />
   <xacro:property name="rolling_moment_coefficient" value="0.0000001" />
-  <!-- Property Blocks -->
+    <!-- Property Blocks -->
   <xacro:property name="body_inertia">
      <inertia ixx="1.657171e-5" ixy="0.830806e-6" ixz="0.718277e-6" iyy="1.6655602e-5" iyz="1.800197e-6" izz="2.9261652e-5" /> <!-- [kg.m^2] [kg.m^2] [kg.m^2] [kg.m^2] [kg.m^2] [kg.m^2] -->
@@ -39,7 +39,7 @@
   <xacro:property name="rotor_inertia">
     <inertia
-    ixx="${1/12 * mass_rotor * (0.006 * 0.006 + 0.001 * 0.001) * rotor_velocity_slowdown_sim}"
-    iyy="${1/12 * mass_rotor * (4 * radius_rotor * radius_rotor + 0.001 * 0.001) * rotor_velocity_slowdown_sim}"
-    izz="${1/12 * mass_rotor * (4 * radius_rotor * radius_rotor + 0.006 * 0.006) * rotor_velocity_slowdown_sim}"
+    ixx="8.33333E-09"
+    iyy="1.08333E-07"
+    izz="1.13333E-07"
     ixy="0.0" ixz="0.0"  iyz="0.0" /> <!-- [kg.m^2] [kg.m^2] [kg.m^2] [kg.m^2] [kg.m^2] [kg.m^2] -->
   </xacro:property>

Commit message: Reduced rotor_velocity_slowdown_sim

File: crazyflie_gazebo/models/rotors_description/urdf/crazyflie.xacro (robot description, xacro)
@@ -8,5 +8,5 @@
   <!-- Properties -->
   <xacro:property name="namespace" value="$(arg namespace)" />
-  <xacro:property name="rotor_velocity_slowdown_sim" value="70" />
+  <xacro:property name="rotor_velocity_slowdown_sim" value="50" />
   <xacro:property name="mesh_file" value="crazyflie.dae" />
   <xacro:property name="mesh_scale" value="1 1 1"/>
@@ -39,7 +39,7 @@
   <xacro:property name="rotor_inertia">
     <inertia
-    ixx="8.33333E-09"
-    iyy="1.08333E-07"
-    izz="1.13333E-07"
+    ixx="${1/12 * mass_rotor * (0.006 * 0.006 + 0.001 * 0.001) * rotor_velocity_slowdown_sim}"
+    iyy="${1/12 * mass_rotor * (4 * radius_rotor * radius_rotor + 0.001 * 0.001) * rotor_velocity_slowdown_sim}"
+    izz="${1/12 * mass_rotor * (4 * radius_rotor * radius_rotor + 0.006 * 0.006) * rotor_velocity_slowdown_sim}"
     ixy="0.0" ixz="0.0"  iyz="0.0" /> <!-- [kg.m^2] [kg.m^2] [kg.m^2] [kg.m^2] [kg.m^2] [kg.m^2] -->
   </xacro:property>

File: crazyflie_gazebo/models/rotors_description/urdf/multirotor_base.xacro (robot description, xacro)
@@ -21,4 +21,17 @@
 <robot xmlns:xacro="http://ros.org/wiki/xacro">
   <!-- Main multirotor link -->
+    <xacro:macro name="box_inertia" params="x y z mass">
+    <inertia ixx="${0.0833333 * mass * (y*y + z*z)}" ixy="0.0" ixz="0.0"
+      iyy="${0.0833333 * mass * (x*x + z*z)}" iyz="0.0"
+      izz="${0.0833333 * mass * (x*x + y*y)}" />
+  </xacro:macro>
+  <!-- Macro for the inertial properties of a box -->
+  <xacro:macro name="box_inertial" params="x y z mass *origin">
+    <inertial>
+      <mass value="${mass}" />
+      <xacro:insert_block name="origin" />
+      <xacro:box_inertia x="${x}" y="${y}" z="${z}" mass="${mass}" />
+    </inertial>
+  </xacro:macro>
   <xacro:macro name="multirotor_base_macro"
     params="robot_namespace mass body_width body_height mesh_file mesh_scale *inertia">

Commit message: trying to send automated commands to the hitl drone. Not sucesful yet

File: crazyflie_gazebo/models/rotors_description/urdf/crazyflie.xacro (robot description, xacro)
@@ -8,5 +8,5 @@
   <!-- Properties -->
   <xacro:property name="namespace" value="$(arg namespace)" />
-  <xacro:property name="rotor_velocity_slowdown_sim" value="50" />
+  <xacro:property name="rotor_velocity_slowdown_sim" value="10" />
   <xacro:property name="mesh_file" value="crazyflie.dae" />
   <xacro:property name="mesh_scale" value="1 1 1"/>

File: crazyflie_gazebo/models/rotors_description/urdf/crazyflie_base.xacro (robot description, xacro)
@@ -48,4 +48,23 @@
     <origin xyz="0 0 0" rpy="0 0 0" />
   </xacro:imu_plugin_macro>
+  <!-- BMI088 IMU -->
+  <!-- <xacro:imu_plugin_macro
+    namespace="${namespace}"
+    imu_suffix=""
+    parent_link="base_link"
+    imu_topic="${imu_topic}"
+    mass_imu_sensor="0.00001"
+    rate="1000"
+    gyroscope_noise_density="2.44e-4"
+    gyroscope_random_walk="4.0e-5"
+    gyroscope_bias_correlation_time="100.0"
+    gyroscope_turn_on_bias_sigma="0.05"
+    accelerometer_noise_density="2.26e-3"
+    accelerometer_random_walk="2.0e-4"
+    accelerometer_bias_correlation_time="300.0"
+    accelerometer_turn_on_bias_sigma="0.2">
+    <inertia ixx="0.0000000001" ixy="0.0" ixz="0.0" iyy="0.0000000001" iyz="0.0" izz="0.0000000001" />
+    <origin xyz="0 0 0" rpy="0 0 0" />
+  </xacro:imu_plugin_macro> -->
 <!--     <xacro:imu_plugin_macro
       namespace="${namespace}"

Commit message: Currently the best version of the simulation working

File: crazyflie_gazebo/models/rotors_description/urdf/crazyflie.xacro (robot description, xacro)
@@ -32,4 +32,6 @@
   <xacro:property name="rotor_drag_coefficient" value="8.06428e-05" />
   <xacro:property name="rolling_moment_coefficient" value="0.0000001" />
+  <xacro:property name="sin45" value="0.707106781186" />
+  <xacro:property name="cos45" value="0.707106781186" />
     <!-- Property Blocks -->
   <xacro:property name="body_inertia">
@@ -38,9 +40,5 @@
   <!-- inertia of a single rotor, assuming it is a cuboid. Height=0.3mm, width=0.9mm -->
   <xacro:property name="rotor_inertia">
-    <inertia
-    ixx="${1/12 * mass_rotor * (0.006 * 0.006 + 0.001 * 0.001) * rotor_velocity_slowdown_sim}"
-    iyy="${1/12 * mass_rotor * (4 * radius_rotor * radius_rotor + 0.001 * 0.001) * rotor_velocity_slowdown_sim}"
-    izz="${1/12 * mass_rotor * (4 * radius_rotor * radius_rotor + 0.006 * 0.006) * rotor_velocity_slowdown_sim}"
-    ixy="0.0" ixz="0.0"  iyz="0.0" /> <!-- [kg.m^2] [kg.m^2] [kg.m^2] [kg.m^2] [kg.m^2] [kg.m^2] -->
+    <xacro:box_inertia x="${radius_rotor}" y="0.007" z="0.003" mass="${mass_rotor*rotor_velocity_slowdown_sim}" />
   </xacro:property>
   <!-- Included URDF Files -->
